Commit message: Restructured the package and optimized URDF

File: mecanum_robot_simulation/urdf/gazeboCamera.xacro (robot description, xacro)
@@ -3,5 +3,5 @@
   <joint name="camera_joint" type="fixed">
       <origin xyz="0.255 0 -0.015" rpy="0 0 0" />
-      <parent link="chasis" />
+      <parent link="base_link" />
       <child link="camera_link" />
   </joint>

File: mecanum_robot_simulation/urdf/gazeboDepthCamera.xacro (robot description, xacro)
@@ -3,5 +3,5 @@
     <joint name="camera_joint" type="fixed">
         <origin xyz="-0.255 0 -0.015" rpy="0 0 ${math.pi}" />
-        <parent link="chasis" />
+        <parent link="base_link" />
         <child link="camera_link" />
     </joint>

File: mecanum_robot_simulation/urdf/gazeboLidar.xacro (robot description, xacro)
@@ -12,5 +12,5 @@
   <joint name="lidar_joint" type="fixed">
       <origin xyz="0 0 0.01" rpy="0 0 0" />
-      <parent link="chasis" />
+      <parent link="base_link" />
       <child link="lidar_frame" />
   </joint>
